File: revisions/XTMT/Feather-RTD.sch (EAGLE design)
At the start: 36 parts, among them U1 MIC5225-3.3, U3 MAX31865, U4 MAX31865, U5 MAX31865, U6 MAX31865

Commit message: Move atributed from page 1 title block to global
Changed lines of the file:
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@@
 <schematic xreflabel="%N (%S.%C%R)" xrefpart="/%S.%C%R">
 <attributes>
+<attribute name="LICENSE" value="CC BY-SA 4.0"/>
+<attribute name="REV" value="XTMT"/>
+<attribute name="TITLE" value="Feather RTD Wing"/>
+<attribute name="URL" value="https://github.com/CapableRobot/Feather-RTD"/>
 </attributes>
 <variantdefs>
@@
 <part name="J1" library="SparkFun-Connectors" library_urn="urn:adsk.eagle:library:513" deviceset="CONN_12" device="NO_SILK" package3d_urn="urn:adsk.eagle:package:38179/1"/>
 <part name="J3" library="SparkFun-Connectors" library_urn="urn:adsk.eagle:library:513" deviceset="CONN_16" device="1X16_NO_SILK" package3d_urn="urn:adsk.eagle:package:38249/1"/>
-<part name="FRAME1" library="CapableRobot" deviceset="LETTER_L" device="">
-<attribute name="LICENSE" value="CC BY-SA 4.0"/>
-<attribute name="REV" value="XTMT"/>
-<attribute name="TITLE" value="Feather RTD Wing"/>
-<attribute name="URL" value="https://github.com/CapableRobot/Feather-RTD"/>
-</part>
+<part name="FRAME1" library="CapableRobot" deviceset="LETTER_L" device=""/>
 <part name="FRAME2" library="CapableRobot" deviceset="LETTER_L" device=""/>
 <part name="FRAME3" library="CapableRobot" deviceset="LETTER_L" device=""/>
@@
 <instance part="J3" gate="G$1" x="83.82" y="45.72" rot="MR0"/>
 <instance part="FRAME1" gate="G$1" x="0" y="0"/>
-<instance part="FRAME1" gate="G$2" x="147.32" y="0">
-<attribute name="REV" x="147.32" y="0" size="1.778" layer="96" display="off"/>
-<attribute name="LICENSE" x="147.32" y="0" size="1.778" layer="96" display="off"/>
-<attribute name="TITLE" x="147.32" y="0" size="1.778" layer="96" display="off"/>
-<attribute name="URL" x="147.32" y="0" size="1.778" layer="96" display="off"/>
-</instance>
+<instance part="FRAME1" gate="G$2" x="147.32" y="0"/>
 <instance part="GND3" gate="1" x="71.12" y="134.62"/>
 <instance part="GND1" gate="1" x="38.1" y="134.62"/>
